File: avs-mod-shield/hardware/avs-mod-shield.kicad_pcb (KiCad board)
At the start: 2 copper layers, 101.6 x 53.3 mm, 13 parts, among them P1 Digital, P10 CONN_1, P11 CONN_1, P12 CONN_1, P13 CONN_1, P2 Power, P3 Analog, P4 Analog, P5 PWM, P6 PWM, P7 Communication, P8 CONN_1, P9 CONN_1

Commit message: continued avs-mod-shield
Parts:
- added XD1: CONN_02X08, Pin_Headers:Pin_Header_Straight_2x08, F.Cu at (174.0, 86.2)
- added XP1: CONN_02X10, Pin_Headers:Pin_Header_Straight_2x10, F.Cu at (107.3, 91.3)
- added XP2: CONN_02X10, Pin_Headers:Pin_Header_Straight_2x10, F.Cu at (117.5, 91.3)
- added XP3: CONN_02X10, Pin_Headers:Pin_Header_Straight_2x10, F.Cu at (127.4, 91.3)
- added XP4: CONN_02X10, Pin_Headers:Pin_Header_Straight_2x10, F.Cu at (137.4, 91.3)
- added XP5: CONN_02X10, Pin_Headers:Pin_Header_Straight_2x10, F.Cu at (147.6, 91.3)
- added XP6: CONN_02X10, Pin_Headers:Pin_Header_Straight_2x10, F.Cu at (157.7, 91.3)
- added XR1: CONN_02X10, Pin_Headers:Pin_Header_Straight_2x10, F.Cu at (187.1, 99.3)
- added XV1: CONN_01X03, Pin_Headers:Pin_Header_Straight_1x03, F.Cu at (115.6, 80.0)
- added XV2: CONN_01X03, Pin_Headers:Pin_Header_Straight_1x03, F.Cu at (121.9, 80.0)
- added XV3: CONN_01X03, Pin_Headers:Pin_Header_Straight_1x03, F.Cu at (128.3, 80.0)
- added XV4: CONN_01X03, Pin_Headers:Pin_Header_Straight_1x03, F.Cu at (134.6, 80.0)
- added XV5: CONN_01X03, Pin_Headers:Pin_Header_Straight_1x03, F.Cu at (141.0, 80.0)
- added XV6: CONN_01X03, Pin_Headers:Pin_Header_Straight_1x03, F.Cu at (147.3, 80.0)
Connections:
- P1 pad 10: /47 -> /AP7
- P1 pad 11: /44 -> /P0
- P1 pad 12: /45 -> /P1
- P1 pad 13: /42 -> /P2
- P1 pad 14: /43 -> /P3
- P1 pad 15: /40 -> /P4
- P1 pad 16: /41 -> /P5
- P1 pad 17: /38 -> /P6
- P1 pad 18: /39 -> /P7
- P1 pad 19: /36 -> (no net)
- P1 pad 20: /37 -> (no net)
- P1 pad 21: /34 -> (no net)
- P1 pad 22: /35 -> (no net)
- P1 pad 23: /32 -> (no net)
- P1 pad 24: /33 -> (no net)
- P1 pad 25: /30 -> (no net)
- P1 pad 26: /31 -> (no net)
- P1 pad 27: /28 -> (no net)
- P1 pad 28: /29 -> (no net)
- P1 pad 29: /26 -> (no net)
- P1 pad 3: /52(SCK) -> /AP0
- P1 pad 30: /27 -> (no net)
- P1 pad 31: /24 -> (no net)
- P1 pad 32: /25 -> (no net)
- P1 pad 33: /22 -> (no net)
- P1 pad 34: /23 -> (no net)
- P1 pad 4: /53(SS) -> /AP1
- P1 pad 5: /50(MISO) -> /AP2
- P1 pad 6: /51(MOSI) -> /AP3
- P1 pad 7: /48 -> /AP4
- P1 pad 8: /49 -> /AP5
- P1 pad 9: /46 -> /AP6
- P10 pad 1: Net-(P10-Pad1) -> (no net)
- P11 pad 1: Net-(P11-Pad1) -> (no net)
- P12 pad 1: Net-(P12-Pad1) -> (no net)
- P13 pad 1: Net-(P13-Pad1) -> (no net)
- P2 pad 1: Net-(P2-Pad1) -> (no net)
- P2 pad 2: /IOREF -> (no net)
- P2 pad 3: /Reset -> (no net)
- P2 pad 4: +3V3 -> (no net)
- P2 pad 8: /Vin -> (no net)
- P3 pad 1: /A0 -> (no net)
- P3 pad 2: /A1 -> (no net)
- P3 pad 3: /A2 -> (no net)
- P3 pad 4: /A3 -> (no net)
- P3 pad 5: /A4 -> (no net)
- P3 pad 6: /A5 -> (no net)
- P3 pad 7: /A6 -> (no net)
- P3 pad 8: /A7 -> (no net)
- P4 pad 1: /A8 -> (no net)
- P4 pad 2: /A9 -> (no net)
- P4 pad 3: /A10 -> (no net)
- P4 pad 4: /A11 -> (no net)
- P4 pad 5: /A12 -> (no net)
- P4 pad 6: /A13 -> (no net)
- P4 pad 7: /A14 -> (no net)
- P4 pad 8: /A15 -> (no net)
- P5 pad 1: /SCL -> (no net)
- P5 pad 10: /8(**) -> (no net)
- P5 pad 2: /SDA -> (no net)
- P5 pad 3: /AREF -> (no net)
- P5 pad 5: /13(**) -> (no net)
- P5 pad 6: /12(**) -> (no net)
- P5 pad 7: /11(**) -> (no net)
- P5 pad 8: /10(**) -> (no net)
- P5 pad 9: /9(**) -> (no net)
- P6 pad 1: /7(**) -> (no net)
- P6 pad 2: /6(**) -> (no net)
- P6 pad 3: /5(**) -> (no net)
- P6 pad 4: /4(**) -> (no net)
- P6 pad 5: /3(**) -> (no net)
- P6 pad 6: /2(**) -> (no net)
- P6 pad 7: /1(Tx0) -> (no net)
- P6 pad 8: /0(Rx0) -> (no net)
- P7 pad 1: /14(Tx3) -> (no net)
- P7 pad 2: /15(Rx3) -> (no net)
- P7 pad 3: /16(Tx2) -> (no net)
- P7 pad 4: /17(Rx2) -> (no net)
- P7 pad 5: /18(Tx1) -> (no net)
- P7 pad 6: /19(Rx1) -> (no net)
- P7 pad 7: /20(SDA) -> (no net)
- P7 pad 8: /21(SCL) -> (no net)
- P8 pad 1: Net-(P8-Pad1) -> (no net)
- P9 pad 1: Net-(P9-Pad1) -> (no net)
Routing:
- net /AP3: track 0.00 -> 105.3 mm
- net /AP7: track 0.00 -> 105.3 mm
- net /AP5: track 0.00 -> 105.3 mm
- net /AP1: track 0.00 -> 105.3 mm
- net /AP4: track 0.00 -> 101.4 mm
- net /AP6: track 0.00 -> 101.2 mm
- net /AP2: track 0.00 -> 100.9 mm
- net /AP0: track 0.00 -> 100.9 mm
- net /P7: track 0.00 -> 95.7 mm
- net /P5: track 0.00 -> 94.5 mm
- net /P1: track 0.00 -> 93.5 mm
- net /P3: track 0.00 -> 92.7 mm
- net /P6: track 0.00 -> 90.2 mm
- net /P4: track 0.00 -> 89.2 mm
- net /P0: track 0.00 -> 87.8 mm
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- added copper zone on B.Cu, net +5V
- added copper zone on F.Cu, net GND
Other:
- net class 0.5 added: clearance 0.2, trace_width 0.5, via_dia 0.6, via_drill 0.4
