File: avs-mod-shield/hardware/avs-mod-shield.sch (KiCad schematic (older format))
At the start: 13 parts, among them P1 Digital, P10 CONN_1, P11 CONN_1, P12 CONN_1, P13 CONN_1, P2 Power, P3 Analog, P4 Analog, P5 PWM, P6 PWM, P7 Communication, P8 CONN_1, P9 CONN_1

Commit message: continued avs-mod-shield
Parts:
- added XD1: CONN_02X08, Pin_Headers:Pin_Header_Straight_2x08, symbol CONN_02X08
- added XP1, XP2, XP3, XP4, XP5, XP6, XR1: CONN_02X10, Pin_Headers:Pin_Header_Straight_2x10, symbol CONN_02X10
- added XV1, XV2, XV3, XV4, XV5, XV6: CONN_01X03, Pin_Headers:Pin_Header_Straight_1x03, symbol CONN_01X03
Connections:
- net labels added: /G, AP0, AP1, AP2, AP3, AP4, AP5, AP6, AP7, LD1, LD2, P0, P1, P2, P3, P4, P5, P6, P7, TA0, TA1, TA2, TA3, TA4, TA5, TA6, TA7, TW0, TW1, TW2, TW3, TW4, TW5, TW6
- net labels removed: 38, 39, 40, 41, 42, 43, 44, 45, 46, 47, 48, 49, 50(MISO), 51(MOSI), 52(SCK), 53(SS)
- wire segments 97 -> 287
Other:
- moved on the sheet: P1
